File: Soyuz.kicad_pcb (KiCad board)
At the start: 2 copper layers, 265.4 x 111.2 mm, 47 parts, among them SW1 SW_Push, U1 ProMicro

Commit message: Updating outlines
Parts:
- removed G***: LOGO, locallib:ai-ring-25mm-mask
- removed O1: Outline, locallib:outline
- added REF**: outline_soyuz, locallib:outline_soyuz, F.Cu at (104.1, 123.2)
Routing:
- removed copper zone on B.Cu, net Earth
- removed copper zone on F.Cu, net Earth
- removed copper zone on B.Cu, net GNDA
- removed copper zone on F.Cu, net GNDA
Other:
- board size 265.4 x 111.2 mm -> 73 x 92.1 mm
- board text removed: "Soyuz Numpad Kit Rev 1.0"
- board text removed: "This is the bottomside of the plate"
- board text removed: "Vendor/Customizing instructions 1. Fork Soyuz on GitHub to create your own copy. Clone onto your PC. 2. Turn your logo into a footprint using bitmap2component, save in locallib.pretty. 3. Place it on the topside of the bottom plate. It is left intentionally blank for this. 4. Alt+3 to render and see if it looks nice. 5. Using the Plot tool, generate the gerbers. The bottom plate is reversible."
