File: Soyuz_bottom.kicad_pcb (KiCad board)
At the start: 2 copper layers, 265.4 x 111.2 mm, 47 parts, among them SW1 SW_Push, U1 ProMicro

Commit message: Created blank bottom plate for acrylic cutting and added dxf export of edge cuts of bottom plate
Parts:
- removed D1, D10, D11, D12, D13, D14, D15, D16, D17, D18, D19, D2, D20, D3, D4, D5, D6, D7, D8, D9: 1N4148, Diodes_THT:D_DO-35_SOD27_P7.62mm_Horizontal
- removed MX1, MX10, MX11, MX12, MX13, MX14, MX15, MX16, MX17, MX19, MX2, MX20, MX21, MX22, MX3, MX4, MX5, MX6, MX7, MX8: MX-1U, MX_Alps_Hybrid:MX-1U-NoLED
- removed MX18, MX23, MX9: MX-2U, MX_Alps_Hybrid:MX-2U-ReversedStabilizers-NoLED
- removed O1: Outline, locallib:outline
- removed SW1: SW_Push, random-keyboard-parts:PushButton_6x6mm_TH_Pretty
- removed U1: ProMicro, promicro:ProMicro-EnforcedTop
- added REF**: outline_bottom, locallib:outline_bottom, F.Cu at (27.9, 133.3)
Routing:
- net ROW4: track 114.9 -> 0.00 mm
- net COL3: track 112.9 -> 0.00 mm
- net COL0: track 99.4 -> 0.00 mm
- net ROW3: track 92.6 -> 0.00 mm
- net COL1: track 91.9 -> 0.00 mm
- net COL2: track 87.5 -> 0.00 mm
- net ROW0: track 85.3 -> 0.00 mm
- net ROW1: track 84.2 -> 0.00 mm
- net GND: track 78.2 -> 0.00 mm
- net ROW2: track 72.7 -> 0.00 mm
- net Net-(SW1-Pad1): track 48.8 -> 0.00 mm
- net Net-(D2-Pad2): track 34.8 -> 0.00 mm
- net Net-(D6-Pad2): track 28.1 -> 0.00 mm
- net Net-(D11-Pad2): track 25.4 -> 0.00 mm
- net Net-(D12-Pad2): track 25.3 -> 0.00 mm
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- added copper zone on B.Cu, net (none)
- added copper zone on F.Cu, net (none)
- removed copper zone on B.Cu, net Earth
- removed copper zone on F.Cu, net Earth
Other:
- board size 265.4 x 111.2 mm -> 92.2 x 111.2 mm
- board text removed: "Pro Micro Component side faces away from PCB"
- board text removed: "Soyuz Numpad Kit Rev 1.0"
- board text removed: "Soyuz PCB R1.0 20190113"
- board text removed: "This is the bottomside of the plate"
- board text removed: "kb.ai03.me"
